File: LEFT_Parade_kicad/LEFT_Parade.kicad_sch (KiCad schematic)
At the start: 23 parts, among them SW1 RotaryEncoder_Switch, SW2 SW_Push, SW3 SW_Push, SW4 SW_Push, SW5 SW_Push, SW6 SW_Push, SW7 SW_Push, SW8 SW_Push, SW9 SW_Push, U1 SeeeduinoXIAO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

Commit message: [Add] game mode
Parts:
- added SW10, SW11, SW12, SW13, SW14, SW15, SW16, SW17: SW_Push_reverse, Button_Switch_Keyboard:SW_Cherry_MX_1.25u_PCB, symbol Switch:SW_Push
- C1, C2: footprint (none) -> Capacitor_THT:C_Axial_L5.1mm_D3.1mm_P7.50mm_Horizontal
- D1, D2, D3, D4, D5, D6, D7, D8: footprint Diode_SMD:D_SOD-323F -> Diode_THT:D_A-405_P7.62mm_Horizontal
- R1, R2: footprint (none) -> Resistor_THT:R_Axial_DIN0207_L6.3mm_D2.5mm_P10.16mm_Horizontal
- SW1: footprint (none) -> Rotary_Encoder:RotaryEncoder_Alps_EC12E-Switch_Vertical_H20mm
- SW2, SW3, SW4, SW5, SW6, SW7, SW8, SW9: footprint (none) -> Button_Switch_Keyboard:SW_Cherry_MX_1.25u_PCB
- U2: footprint (none) -> Package_DIP:CERDIP-16_W7.62mm_SideBrazed
Connections:
- net at SW5.1, SW9.1, U2.12 (~{Q0}): now also SW13.1, SW17.1
- net at D4.1 (K), SW5.2: now also SW13.2
- net at D8.1 (K), SW9.2: now also SW17.2
- net at SW4.1, SW8.1, U2.11 (~{Q1}): now also SW12.1, SW16.1
- net at D3.1 (K), SW4.2: now also SW12.2
- net at SW3.1, SW7.1, U2.10 (~{Q2}): now also SW11.1, SW15.1
- net at D6.1 (K), SW7.2: now also SW15.2
- net at D5.1 (K), SW6.2: now also SW14.2
- net at D7.1 (K), SW8.2: now also SW16.2
- net at SW2.1, SW6.1, U2.9 (~{Q3}): now also SW10.1, SW14.1
- net at D2.1 (K), SW3.2: now also SW11.2
- net at D1.1 (K), SW2.2: now also SW10.2
