File: LEFT_Parade_kicad/LEFT_Parade.kicad_pcb (KiCad board)
At the start: 2 copper layers, 83.5 x 72.5 mm, 34 parts, among them SW1 RotaryEncoder_Switch, SW10 SW_Push_reverse, SW11 SW_Push_reverse, SW12 SW_Push_reverse, SW13 SW_Push_reverse, SW14 SW_Push_reverse, SW15 SW_Push_reverse, SW16 SW_Push_reverse, SW17 SW_Push_reverse, SW2 SW_Push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

Commit message: [Modify] Readme.md
Parts:
- added ?: , , F.Cu at (43.5, 36.0)
- added ?: , , F.Cu at (44.0, 102.5)
- added ?: , , F.Cu at (124.5, 102.0)
- added G***: LOGO, illust:normaltype_bit, F.Cu at (54.0, 98.5)
- added G***: LOGO, illust:normaltype_bit_reverse, F.Cu at (86.0, 98.5)
- added REF**: MountingHole_3.2mm_M3, MountingHole:MountingHole_3.2mm_M3, F.Cu at (124.0, 36.0)
- moved SW12 0.08 mm to (73.0, 41.0)
- moved SW14 0.08 mm to (113.0, 61.0)
- moved SW3 0.08 mm to (75.5, 38.4)
- moved SW9 0.08 mm to (115.5, 58.4)
Routing:
- net Net-(U2B-~{Q2}): track 79.2 -> 97.3 mm
- net Net-(D1-K): track 86.8 -> 101.0 mm
- net Net-(D8-K): track 57.5 -> 70.5 mm
- net Net-(U2B-~{Q3}): track 114.4 -> 123.2 mm
- net Net-(D7-K): track 14.5 -> 22.1 mm
- net Net-(D4-K): track 57.7 -> 65.4 mm
- net Net-(D5-K): track 92.2 -> 85.2 mm
- net Net-(D6-K): track 41.9 -> 48.9 mm
- net Net-(D3-K): track 16.5 -> 22.2 mm
- net Net-(U2B-~{Q1}): track 79.5 -> 83.6 mm
- net Net-(D1-A): track 92.3 -> 94.1 mm, vias 1 -> 0
- net Net-(U2B-~{Q0}): track 118.4 -> 119.0 mm
Other:
- board size 83.5 x 72.5 mm -> 86 x 72.5 mm
- board text added: "LEFT Parade"
- board text added: "RIGHT Parade"

Commit message: [Modify] Version UP
Parts:
- removed R2: 10kΩ, Resistor_THT:R_Axial_DIN0207_L6.3mm_D2.5mm_P10.16mm_Horizontal
- added D11: LED, LED_THT:LED_D3.0mm_Clear, F.Cu at (75.0, 95.0)
- R1: value 10kΩ -> 1k
- moved D10 6.14 mm to (68.7, 95.0)
- moved D9 6.04 mm to (62.7, 95.0)
- moved R1 5.96 mm to (81.3, 92.0)
Connections:
- C1 pad 1: Net-(C1-Pad1) -> Net-(U2A-GND)
- C1 pad 2: Net-(C1-Pad2) -> Net-(U1-PA11_A3_D3)
- C2 pad 1: Net-(C2-Pad1) -> Net-(U1-PA8_A4_D4_SDA)
- C2 pad 2: Net-(C1-Pad1) -> Net-(U2A-GND)
- C3 pad 1: Net-(U1-PA5_A9_D9_MISO) -> Net-(U2A-GND)
- R1 pad 1: Net-(U1-PA8_A4_D4_SDA) -> Net-(U1-3V3)
- R1 pad 2: Net-(C2-Pad1) -> Net-(D10-A)
- SW1 pad A: Net-(C2-Pad1) -> Net-(U1-PA8_A4_D4_SDA)
- SW1 pad B: Net-(C1-Pad2) -> Net-(U1-PA11_A3_D3)
- SW1 pad C: Net-(C1-Pad1) -> Net-(U2A-GND)
- SW1 pad S1: Net-(U1-PA5_A9_D9_MISO) -> Net-(U2A-GND)
- U1 pad 11: Net-(U1-PA5_A9_D9_MISO) -> Net-(U1-PA6_A10_D10_MOSI)
- U1 pad 13: Net-(U1-PA5_A9_D9_MISO) -> Net-(U2A-GND)
- U1 pad 14: Net-(D10-A) -> unconnected-(U1-5V-Pad14)
- U2 pad 1: Net-(U1-PA5_A9_D9_MISO) -> Net-(U2A-GND)
- U2 pad 13: Net-(U1-PA5_A9_D9_MISO) -> Net-(U1-PA6_A10_D10_MOSI)
- U2 pad 15: Net-(U1-PA5_A9_D9_MISO) -> Net-(U2A-GND)
- U2 pad 4: unconnected-(U2A-~{Q0}-Pad4) -> Net-(D11-K)
- U2 pad 8: Net-(U1-PA5_A9_D9_MISO) -> Net-(U2A-GND)
Routing:
- net Net-(U2A-GND): track 0.00 -> 156.6 mm
- net Net-(U1-PA5_A9_D9_MISO): track 103.3 -> 17.6 mm
- net Net-(U1-PA8_A4_D4_SDA): track 23.7 -> 91.8 mm
- net Net-(U1-PA6_A10_D10_MOSI): track 0.00 -> 46.4 mm
- net Net-(C1-Pad1): track 43.8 -> 0.00 mm
- net Net-(C2-Pad1): track 42.5 -> 0.00 mm
- net Net-(U1-PA11_A3_D3): track 40.6 -> 82.4 mm
- net Net-(U1-3V3): track 15.0 -> 42.9 mm
- net Net-(C1-Pad2): track 20.8 -> 0.00 mm
- net Net-(D11-K): track 0.00 -> 20.3 mm
- net Net-(D10-A): track 39.0 -> 31.3 mm, vias 1 -> 0
- net Net-(D10-K): track 7.14 -> 13.8 mm
- net Net-(D9-K): track 19.8 -> 25.6 mm
- added copper zone on B.Cu, net Net-(U2A-GND)
- added copper zone on F.Cu, net Net-(U2A-GND)
Other:
- board text added: "ver. 0.1.2"
